File: schem/displaywriter-usb.kicad_pcb (KiCad board)
At the start: 2 copper layers, 119.8 x 32.5 mm, 92 parts, among them CON1 USB-MINI-B, P2 CONN_3X2, P3 Chassis GND, SW1 PROG, SW2 RESET, U1 ATMEGA32U2, U2 DAC101S101, U3 LM339A, U4 LM339A, U5 74AHC595, U6 74AHC595, X1 16MHz

Commit message: 0.6.6
Parts:
- R7: value 47K -> 4.7K
- R8: value 10K -> 1K
- SW1: value PROG -> SW_PUSH
- SW2: value RESET -> SW_PUSH
Changed lines of the file:
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@@
       (effects (font (size 0.4 0.4) (thickness 0.1)) (justify mirror))
     )
-    (fp_text value RESET (at -1.75 0 180) (layer B.SilkS)
+    (fp_text value SW_PUSH (at -1.75 0 180) (layer B.SilkS)
       (effects (font (size 0.4 0.4) (thickness 0.1)) (justify mirror))
     )
@@
       (effects (font (size 0.4 0.4) (thickness 0.1)) (justify mirror))
     )
-    (fp_text value PROG (at -1.78 -0.1 180) (layer B.SilkS)
+    (fp_text value SW_PUSH (at -1.78 -0.1 180) (layer B.SilkS)
       (effects (font (size 0.4 0.4) (thickness 0.1)) (justify mirror))
     )
@@
       (effects (font (size 0.50038 0.50038) (thickness 0.10922)))
     )
-    (fp_text value 47K (at 0 0 360) (layer F.SilkS)
+    (fp_text value 4.7K (at 0 0 360) (layer F.SilkS)
       (effects (font (size 0.50038 0.50038) (thickness 0.10922)))
     )
@@
       (effects (font (size 0.50038 0.50038) (thickness 0.10922)))
     )
-    (fp_text value 10K (at 0 0 360) (layer F.SilkS)
-      (effects (font (size 0.50038 0.50038) (thickness 0.10922)))
-    )
+    (fp_text value 1K (at 0 0 360) (layer F.SilkS)
+      (effects (font (size 0.50038 0.50038) (thickness 0.10922)))
+    )
