File: schem/displaywriter-usb.sch (KiCad schematic (older format))
At the start: 38 parts, among them CON1 USB-MINI-B, P2 CONN_3X2, P3 Chassis GND, SW1 SW_PUSH, SW2 SW_PUSH, U1 ATMEGA32U2, U2 DAC101S101, U3 LM339A, U4 LM339A, U5 74AHC595, U6 74AHC595, X1 16MHz

Commit message: 0.6.6
Parts:
- R7: value 47K -> 4.7K
- R8: value 10K -> 1K
Changed lines of the file:
@@
 Sheet 1 1
 Title ""
-Date "15 apr 2014"
+Date "11 may 2014"
 Rev ""
 Comp ""
@@
 P 11800 8750
 F 0 "R7" V 11880 8750 40  0000 C CNN
-F 1 "47K" V 11807 8751 40  0000 C CNN
+F 1 "4.7K" V 11807 8751 40  0000 C CNN
 F 2 "~" V 11730 8750 30  0000 C CNN
 F 3 "~" H 11800 8750 30  0000 C CNN
@@
 P 11800 9350
 F 0 "R8" V 11880 9350 40  0000 C CNN
-F 1 "10K" V 11807 9351 40  0000 C CNN
+F 1 "1K" V 11807 9351 40  0000 C CNN
 F 2 "~" V 11730 9350 30  0000 C CNN
 F 3 "~" H 11800 9350 30  0000 C CNN
