File: schem/model-f-usb.sch (KiCad schematic (older format))
At the start: 43 parts, among them P1 CONN_5, P2 CONN_3X2, P3 Chassis GND, P4 Chassis GND, P5 Chassis GND, P6 Chassis GND, P7 Chassis GND, P8 Chassis GND, SW1 SW_PUSH, SW2 SW_PUSH, U1 ATMEGA32U2, U2 DAC101S101, U3 LM339A, U4 LM339A, U5 74AHC595, U6 74AHC595, X1 16MHz

Commit message: 0.6.7, imported from xwhatit's untracked source code
Parts:
- removed P1: CONN_5, ~, symbol CONN_5
- removed P3, P4, P5, P6, P7, P8: Chassis GND, ~, symbol CONN_1
- added P1: USB, ~, symbol USB-MINI-B
- SW1: value SW_PUSH -> PROG
- SW2: value SW_PUSH -> RESET
Connections:
- wire segments 263 -> 255
- no-connect marks 3 -> 7
Other:
- moved on the sheet: C6
