File: schem/model-f-3178-adaptor.kicad_pcb (KiCad board)
At the start: 2 copper layers, 127 x 6.5 mm, 2 parts

Commit message: 0.7.0, imported from xwhatits untracked repository
Parts:
- PMF2: footprint PIN_ARRAY_3_96-30X1 -> PIN_ARRAY_3_96-30X1_large_pads
Other:
- board text added: "Model-F-3178-Adaptor Rev1 2014-05-23 Tom Wong-Cornall"
- board text removed: "Model-F-3178-Adaptor Rev1 2014-05-12 Tom Wong-Cornall"
Changed lines of the file:
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@@
     (links 35)
     (no_connects 0)
-    (area 146.410478 137.600199 274.672855 144.399801)
+    (area 146.720199 137.600199 274.672855 144.539725)
     (thickness 1.6)
     (drawings 7)
@@
     (pad_to_mask_clearance 0)
     (aux_axis_origin 0 0)
-    (visible_elements FFFFFBFF)
+    (visible_elements 7FFFFFFF)
     (pcbplotparams
       (layerselection 284196865)
@@
     )
   )
-  (module PIN_ARRAY_3_96-30X1 (layer F.Cu)
+  (module PIN_ARRAY_3_96-30X1_large_pads   locked (layer F.Cu)
     (at 206.5 142.75)
-    (fp_text reference PMF2 (at -58.75 0.01 90) (layer F.SilkS)
-      (effects (font (size 0.5 0.5) (thickness 0.125)))
-    )
-    (fp_text value Kbd-3178 (at -57.5 -1.74) (layer F.SilkS)
-      (effects (font (size 0.5 0.5) (thickness 0.125)))
+    (fp_text reference PMF2 (at 0 -2) (layer F.SilkS)
+      (effects (font (size 1.016 1.016) (thickness 0.2032)))
+    )
+    (fp_text value Kbd-3178 (at 0 0) (layer F.SilkS) hide
+      (effects (font (size 1.016 0.889) (thickness 0.2032)))
     )
     (fp_line (start -55.44 -1.27) (end -55.44 1.27) (layer F.SilkS) (width 0.15))
@@
     (fp_line (start 59.4 1.27) (end 59.4 -1.27) (layer F.SilkS) (width 0.15))
     (fp_line (start 59.4 -1.27) (end -59.4 -1.27) (layer F.SilkS) (width 0.15))
-    (pad 1 thru_hole rect (at -57.42 0) (size 1.524 1.524) (drill 1.016)
-      (layers *.Cu *.Mask F.SilkS)
-      (net 1 GND)
-      (zone_connect 1)
-      (thermal_width 0.508)
-      (thermal_gap 0.508)
-    )
-    (pad 2 thru_hole circle (at -53.46 0) (size 1.524 1.524) (drill 1.016)
-      (layers *.Cu *.Mask F.SilkS)
-      (net 1 GND)
-      (zone_connect 1)
-      (thermal_width 0.508)
-      (thermal_gap 0.508)
-    )
-    (pad 3 thru_hole circle (at -49.5 0) (size 1.524 1.524) (drill 1.016)
-      (layers *.Cu *.Mask F.SilkS)
-      (net 1 GND)
-    )
-    (pad 4 thru_hole circle (at -45.54 0) (size 1.524 1.524) (drill 1.016)
-      (layers *.Cu *.Mask F.SilkS)
-      (net 1 GND)
-    )
-    (pad 5 thru_hole circle (at -41.58 0) (size 1.524 1.524) (drill 1.016)
-      (layers *.Cu *.Mask F.SilkS)
-      (net 1 GND)
-    )
-    (pad 6 thru_hole circle (at -37.62 0) (size 1.524 1.524) (drill 1.016)
-      (layers *.Cu *.Mask F.SilkS)
-      (net 1 GND)
-    )
-    (pad 7 thru_hole circle (at -33.66 0) (size 1.524 1.524) (drill 1.016)
-      (layers *.Cu *.Mask F.SilkS)
-      (net 1 GND)
-    )
-    (pad 8 thru_hole circle (at -29.7 0) (size 1.524 1.524) (drill 1.016)
-      (layers *.Cu *.Mask F.SilkS)
-      (net 1 GND)
-    )
-    (pad 9 thru_hole circle (at -25.74 0) (size 1.524 1.524) (drill 1.016)
-      (layers *.Cu *.Mask F.SilkS)
-      (net 1 GND)
-    )
-    (pad 10 thru_hole circle (at -21.78 0) (size 1.524 1.524) (drill 1.016)
+    (pad 1 thru_hole rect (at -57.42 0) (size 2.1 2.1) (drill 1.6)
+      (layers *.Cu *.Mask F.SilkS)
+      (net 1 GND)
+      (zone_connect 1)
+      (thermal_width 0.508)
+      (thermal_gap 0.508)
+    )
+    (pad 2 thru_hole circle (at -53.46 0) (size 2.1 2.1) (drill 1.6)
+      (layers *.Cu *.Mask F.SilkS)
+      (net 1 GND)
+      (zone_connect 1)
+      (thermal_width 0.508)
+      (thermal_gap 0.508)
+    )
+    (pad 3 thru_hole circle (at -49.5 0) (size 2.1 2.1) (drill 1.6)
+      (layers *.Cu *.Mask F.SilkS)
+      (net 1 GND)
+    )
+    (pad 4 thru_hole circle (at -45.54 0) (size 2.1 2.1) (drill 1.6)
+      (layers *.Cu *.Mask F.SilkS)
+      (net 1 GND)
+    )
+    (pad 5 thru_hole circle (at -41.58 0) (size 2.1 2.1) (drill 1.6)
+      (layers *.Cu *.Mask F.SilkS)
+      (net 1 GND)
+    )
+    (pad 6 thru_hole circle (at -37.62 0) (size 2.1 2.1) (drill 1.6)
+      (layers *.Cu *.Mask F.SilkS)
+      (net 1 GND)
+    )
+    (pad 7 thru_hole circle (at -33.66 0) (size 2.1 2.1) (drill 1.6)
+      (layers *.Cu *.Mask F.SilkS)
+      (net 1 GND)
+    )
+    (pad 8 thru_hole circle (at -29.7 0) (size 2.1 2.1) (drill 1.6)
+      (layers *.Cu *.Mask F.SilkS)
+      (net 1 GND)
+    )
+    (pad 9 thru_hole circle (at -25.74 0) (size 2.1 2.1) (drill 1.6)
+      (layers *.Cu *.Mask F.SilkS)
+      (net 1 GND)
+    )
+    (pad 10 thru_hole circle (at -21.78 0) (size 2.1 2.1) (drill 1.6)
       (layers *.Cu *.Mask F.SilkS)
       (net 12 N-0000021)
     )
-    (pad 11 thru_hole circle (at -17.82 0) (size 1.524 1.524) (drill 1.016)
+    (pad 11 thru_hole circle (at -17.82 0) (size 2.1 2.1) (drill 1.6)
       (layers *.Cu *.Mask F.SilkS)
       (net 15 N-0000024)
@@
       (thermal_gap 0.508)
     )
-    (pad 12 thru_hole circle (at -13.86 0) (size 1.524 1.524) (drill 1.016)
+    (pad 12 thru_hole circle (at -13.86 0) (size 2.1 2.1) (drill 1.6)
       (layers *.Cu *.Mask F.SilkS)
       (net 14 N-0000023)
@@
       (thermal_gap 0.508)
     )
-    (pad 13 thru_hole circle (at -9.9 0) (size 1.524 1.524) (drill 1.016)
+    (pad 13 thru_hole circle (at -9.9 0) (size 2.1 2.1) (drill 1.6)
       (layers *.Cu *.Mask F.SilkS)
       (net 13 N-0000022)
     )
-    (pad 14 thru_hole circle (at -5.94 0) (size 1.524 1.524) (drill 1.016)
+    (pad 14 thru_hole circle (at -5.94 0) (size 2.1 2.1) (drill 1.6)
       (layers *.Cu *.Mask F.SilkS)
       (net 21 N-000007)
     )
-    (pad 15 thru_hole circle (at -1.98 0) (size 1.524 1.524) (drill 1.016)
+    (pad 15 thru_hole circle (at -1.98 0) (size 2.1 2.1) (drill 1.6)
       (layers *.Cu *.Mask F.SilkS)
       (net 20 N-000006)
     )
-    (pad 16 thru_hole circle (at 1.98 0) (size 1.524 1.524) (drill 1.016)
+    (pad 16 thru_hole circle (at 1.98 0) (size 2.1 2.1) (drill 1.6)
       (layers *.Cu *.Mask F.SilkS)
       (net 19 N-000005)
     )
-    (pad 17 thru_hole circle (at 5.94 0) (size 1.524 1.524) (drill 1.016)
+    (pad 17 thru_hole circle (at 5.94 0) (size 2.1 2.1) (drill 1.6)
       (layers *.Cu *.Mask F.SilkS)
       (net 2 N-000001)
     )
-    (pad 18 thru_hole circle (at 9.9 0) (size 1.524 1.524) (drill 1.016)
+    (pad 18 thru_hole circle (at 9.9 0) (size 2.1 2.1) (drill 1.6)
       (layers *.Cu *.Mask F.SilkS)
       (net 18 N-000004)
     )
-    (pad 19 thru_hole circle (at 13.86 0) (size 1.524 1.524) (drill 1.016)
+    (pad 19 thru_hole circle (at 13.86 0) (size 2.1 2.1) (drill 1.6)
       (layers *.Cu *.Mask F.SilkS)
       (net 17 N-000003)
     )
-    (pad 20 thru_hole circle (at 17.82 0) (size 1.524 1.524) (drill 1.016)
+    (pad 20 thru_hole circle (at 17.82 0) (size 2.1 2.1) (drill 1.6)
       (layers *.Cu *.Mask F.SilkS)
       (net 10 N-000002)
     )
-    (pad 21 thru_hole circle (at 21.78 0) (size 1.524 1.524) (drill 1.016)
+    (pad 21 thru_hole circle (at 21.78 0) (size 2.1 2.1) (drill 1.6)
       (layers *.Cu *.Mask F.SilkS)
       (net 3 N-0000013)
     )
-    (pad 22 thru_hole circle (at 25.74 0) (size 1.524 1.524) (drill 1.016)
-      (layers *.Cu *.Mask F.SilkS)
-      (net 1 GND)
-    )
-    (pad 23 thru_hole circle (at 29.7 0) (size 1.524 1.524) (drill 1.016)
+    (pad 22 thru_hole circle (at 25.74 0) (size 2.1 2.1) (drill 1.6)
+      (layers *.Cu *.Mask F.SilkS)
+      (net 1 GND)
+    )
+    (pad 23 thru_hole circle (at 29.7 0) (size 2.1 2.1) (drill 1.6)
       (layers *.Cu *.Mask F.SilkS)
       (net 16 N-0000025)
     )
-    (pad 24 thru_hole circle (at 33.66 0) (size 1.524 1.524) (drill 1.016)
+    (pad 24 thru_hole circle (at 33.66 0) (size 2.1 2.1) (drill 1.6)
       (layers *.Cu *.Mask F.SilkS)
       (net 4 N-0000014)
     )
-    (pad 25 thru_hole circle (at 37.62 0) (size 1.524 1.524) (drill 1.016)
+    (pad 25 thru_hole circle (at 37.62 0) (size 2.1 2.1) (drill 1.6)
       (layers *.Cu *.Mask F.SilkS)
       (net 5 N-0000015)
     )
-    (pad 26 thru_hole circle (at 41.58 0) (size 1.524 1.524) (drill 1.016)
+    (pad 26 thru_hole circle (at 41.58 0) (size 2.1 2.1) (drill 1.6)
       (layers *.Cu *.Mask F.SilkS)
       (net 6 N-0000016)
     )
-    (pad 27 thru_hole circle (at 45.54 0) (size 1.524 1.524) (drill 1.016)
+    (pad 27 thru_hole circle (at 45.54 0) (size 2.1 2.1) (drill 1.6)
       (layers *.Cu *.Mask F.SilkS)
       (net 7 N-0000017)
     )
-    (pad 28 thru_hole circle (at 49.5 0) (size 1.524 1.524) (drill 1.016)
+    (pad 28 thru_hole circle (at 49.5 0) (size 2.1 2.1) (drill 1.6)
       (layers *.Cu *.Mask F.SilkS)
       (net 8 N-0000018)
     )
-    (pad 29 thru_hole circle (at 53.46 0) (size 1.524 1.524) (drill 1.016)
+    (pad 29 thru_hole circle (at 53.46 0) (size 2.1 2.1) (drill 1.6)
       (layers *.Cu *.Mask F.SilkS)
       (net 9 N-0000019)
@@
       (thermal_gap 0.508)
     )
-    (pad 30 thru_hole circle (at 57.42 0) (size 1.524 1.524) (drill 1.016)
+    (pad 30 thru_hole circle (at 57.42 0) (size 2.1 2.1) (drill 1.6)
       (layers *.Cu *.Mask F.SilkS)
       (net 11 N-0000020)
@@
   (gr_line (start 147 144) (end 147 144.25) (angle 90) (layer Edge.Cuts) (width 0.1))
   (gr_line (start 147 137.75) (end 147 138.25) (angle 90) (layer Edge.Cuts) (width 0.1))
-  (gr_text "Model-F-3178-Adaptor\nRev1 2014-05-12\nTom Wong-Cornall\n" (at 273.5 141.75) (layer F.SilkS)
+  (gr_text "Model-F-3178-Adaptor\nRev1 2014-05-23\nTom Wong-Cornall\n" (at 273.5 141.75) (layer F.SilkS)
     (effects (font (size 0.4 0.4) (thickness 0.1)) (justify right))
   )
