File: schem/solenoid-driver.kicad_pcb (KiCad board)
At the start: 2 copper layers, 45.2 x 21.2 mm, 22 parts, among them P1 CONN_3X2, P2 TST, P3 CONN_2, P4 Chassis GND, U1 MIC2009A-1, U2 ULN2003, U3 MIC2250-2

Commit message: 0.6.2
Parts:
- removed C7: 220uF, c_elec_6.3x7.7
- removed P2: TST, TP
- added R6: 100K, SM0805, F.Cu at (216.5, 145.5)
- moved R2 2.37 mm to (216.5, 143.2)
- moved R1 1.00 mm to (212.5, 145.5)
Connections:
- R2 pad 2: N-000003 -> N-0000012
- U1 pad 4: N-000003 -> N-0000012
- U3 pad 4: /+5V_Gated -> N-0000012
Routing:
- net N-0000012: track 0.00 -> 21.5 mm
- net N-000003: track 10.6 -> 0.00 mm
- net /+5V_Gated: track 27.0 -> 18.8 mm
- net GND: track 89.8 -> 93.9 mm
- net N-000007: track 5.66 -> 8.44 mm
- net +5V: track 16.4 -> 18.6 mm
Other:
- board text added: "Beamspring-USB Solenoid Driver Rev2 2014-05-10 Tom Wong-Cornall"
- board text removed: "Beamspring-USB Solenoid Driver Rev1 2014-04-06 Tom Wong-Cornall"

Commit message: 0.8.0, imported from xwhatits untracked repository
Parts:
- D1: value 1N5819 -> B220A; footprint DO-41 -> DO214AC_SMA; moved to F.Cu
- D2: value LED -> Actuating; footprint SM1206POL -> LED-0603
- moved D1 5.05 mm to (192.5, 146.8), turned to 270 degrees
- moved R4 4.12 mm to (195.0, 155.5)
- moved R5 4.03 mm to (198.5, 155.5)
- moved C5 2.50 mm to (194.0, 152.5)
- moved C6 1.99 mm to (186.8, 146.0), turned to 270 degrees
- moved D2 1.82 mm to (187.0, 139.8)
- moved P4 1.77 mm to (178.5, 140.8)
- moved R3 1.03 mm to (189.8, 140.8), turned to 270 degrees
Routing:
- net GND: track 93.9 -> 127.8 mm, vias 9 -> 20
- net +9V: track 29.2 -> 10.9 mm
- net N-0000013: track 9.51 -> 4.93 mm
- net /SW: track 11.5 -> 8.95 mm
- net N-000008: track 18.8 -> 17.1 mm
- net N-000009: track 2.52 -> 2.02 mm
Other:
- outline, holes or cut-outs redrawn
- board text added: "Beamspring USB Solenoid Driver"
- board text added: "Rev3 20140811"
- board text added: "Tom Wong-Cornall"
- board text removed: "Beamspring-USB Solenoid Driver Rev2 2014-05-10 Tom Wong-Cornall"
