File: schem/solenoid-driver.sch (KiCad schematic (older format))
At the start: 22 parts, among them P1 CONN_3X2, P2 TST, P3 CONN_2, P4 Chassis GND, U1 MIC2009A-1, U2 ULN2003, U3 MIC2250-2

Commit message: 0.6.2
Parts:
- removed C7: 220uF, ~, symbol CP
- removed P2: TST, ~, symbol TST
- added R6: 100K, ~, symbol R
Connections:
- wire segments 63 -> 66
Other:
- moved on the sheet: C1, C2, R2
Changed lines of the file:
@@
 Sheet 1 1
 Title "noname.sch"
-Date "6 apr 2014"
+Date "10 may 2014"
 Rev ""
 Comp ""
@@
 L C C2
 U 1 1 533DEA52
-P 3000 2700
-F 0 "C2" H 3000 2800 40  0000 L CNN
-F 1 "0.1uF" H 3006 2615 40  0000 L CNN
-F 2 "~" H 3038 2550 30  0000 C CNN
-F 3 "~" H 3000 2700 60  0000 C CNN
-	1    3000 2700
+P 2450 2700
+F 0 "C2" H 2450 2800 40  0000 L CNN
+F 1 "0.1uF" H 2456 2615 40  0000 L CNN
+F 2 "~" H 2488 2550 30  0000 C CNN
+F 3 "~" H 2450 2700 60  0000 C CNN
+	1    2450 2700
 	1    0    0    -1
 $EndComp
@@
 L GND #PWR05
 U 1 1 533F902C
-P 2850 3000
-F 0 "#PWR05" H 2850 3000 30  0001 C CNN
-F 1 "GND" H 2850 2930 30  0001 C CNN
-F 2 "" H 2850 3000 60  0000 C CNN
-F 3 "" H 2850 3000 60  0000 C CNN
-	1    2850 3000
+P 2300 3000
+F 0 "#PWR05" H 2300 3000 30  0001 C CNN
+F 1 "GND" H 2300 2930 30  0001 C CNN
+F 2 "" H 2300 3000 60  0000 C CNN
+F 3 "" H 2300 3000 60  0000 C CNN
+	1    2300 3000
 	1    0    0    -1
 $EndComp
@@
 $EndComp
 $Comp
-L TST P2
-U 1 1 533F956A
-P 4850 2850
-F 0 "P2" H 4850 3150 40  0000 C CNN
-F 1 "TST" H 4850 3100 30  0000 C CNN
-F 2 "~" H 4850 2850 60  0000 C CNN
-F 3 "~" H 4850 2850 60  0000 C CNN
-	1    4850 2850
-	-1   0    0    1
-$EndComp
-$Comp
 L R R2
 U 1 1 533F9579
-P 5200 2750
-F 0 "R2" V 5280 2750 40  0000 C CNN
-F 1 "100K" V 5207 2751 40  0000 C CNN
-F 2 "~" V 5130 2750 30  0000 C CNN
-F 3 "~" H 5200 2750 30  0000 C CNN
-	1    5200 2750
-	0    1    1    0
+P 5450 3050
+F 0 "R2" V 5530 3050 40  0000 C CNN
+F 1 "100K" V 5457 3051 40  0000 C CNN
+F 2 "~" V 5380 3050 30  0000 C CNN
+F 3 "~" H 5450 3050 30  0000 C CNN
+	1    5450 3050
+	1    0    0    -1
 $EndComp
 $Comp
@@
 L C C1
 U 1 1 533F9B5C
-P 2700 2700
-F 0 "C1" H 2700 2800 40  0000 L CNN
-F 1 "1uF" H 2706 2615 40  0000 L CNN
-F 2 "~" H 2738 2550 30  0000 C CNN
-F 3 "~" H 2700 2700 60  0000 C CNN
-	1    2700 2700
+P 2150 2700
+F 0 "C1" H 2150 2800 40  0000 L CNN
+F 1 "1uF" H 2156 2615 40  0000 L CNN
+F 2 "~" H 2188 2550 30  0000 C CNN
+F 3 "~" H 2150 2700 60  0000 C CNN
+	1    2150 2700
 	1    0    0    -1
 $EndComp
@@
 L +5V #PWR08
 U 1 1 533F9C87
-P 2850 2400
-F 0 "#PWR08" H 2850 2490 20  0001 C CNN
-F 1 "+5V" H 2850 2490 30  0000 C CNN
-F 2 "" H 2850 2400 60  0000 C CNN
-F 3 "" H 2850 2400 60  0000 C CNN
-	1    2850 2400
+P 2300 2400
+F 0 "#PWR08" H 2300 2490 20  0001 C CNN
+F 1 "+5V" H 2300 2490 30  0000 C CNN
+F 2 "" H 2300 2400 60  0000 C CNN
+F 3 "" H 2300 2400 60  0000 C CNN
+	1    2300 2400
 	1    0    0    -1
 $EndComp
@@
 $EndComp
 $Comp
-L CP C7
-U 1 1 5340A587
-P 5800 2850
-F 0 "C7" H 5850 2950 40  0000 L CNN
-F 1 "220uF" H 5850 2750 40  0000 L CNN
-F 2 "~" H 5900 2700 30  0000 C CNN
-F 3 "~" H 5800 2850 300 0000 C CNN
-	1    5800 2850
-	1    0    0    -1
-$EndComp
-$Comp
-L GND #PWR017
-U 1 1 5340A693
-P 5800 3050
-F 0 "#PWR017" H 5800 3050 30  0001 C CNN
-F 1 "GND" H 5800 2980 30  0001 C CNN
-F 2 "" H 5800 3050 60  0000 C CNN
-F 3 "" H 5800 3050 60  0000 C CNN
-	1    5800 3050
-	1    0    0    -1
-$EndComp
-$Comp
-L +9V #PWR018
+L +9V #PWR017
 U 1 1 5340AEE5
 P 8950 2500
-F 0 "#PWR018" H 8950 2470 20  0001 C CNN
+F 0 "#PWR017" H 8950 2470 20  0001 C CNN
 F 1 "+9V" H 8950 2610 30  0000 C CNN
 F 2 "" H 8950 2500 60  0000 C CNN
@@
 $EndComp
 $Comp
-L +9V #PWR019
+L +9V #PWR018
 U 1 1 5340AEF4
 P 6700 4700
-F 0 "#PWR019" H 6700 4670 20  0001 C CNN
+F 0 "#PWR018" H 6700 4670 20  0001 C CNN
 F 1 "+9V" H 6700 4810 30  0000 C CNN
 F 2 "" H 6700 4700 60  0000 C CNN
@@
 $EndComp
 $Comp
-L +9V #PWR020
+L +9V #PWR019
 U 1 1 5340AF03
 P 7300 4300
-F 0 "#PWR020" H 7300 4270 20  0001 C CNN
+F 0 "#PWR019" H 7300 4270 20  0001 C CNN
 F 1 "+9V" H 7300 4410 30  0000 C CNN
 F 2 "" H 7300 4300 60  0000 C CNN
@@
 $EndComp
 $Comp
-L +9V #PWR021
+L +9V #PWR020
 U 1 1 5340B0FB
 P 6350 5050
-F 0 "#PWR021" H 6350 5020 20  0001 C CNN
+F 0 "#PWR020" H 6350 5020 20  0001 C CNN
 F 1 "+9V" H 6350 5160 30  0000 C CNN
 F 2 "" H 6350 5050 60  0000 C CNN
@@
 	3200 2550 3350 2550
 Wire Wire Line
-	2700 2450 3200 2450
-Wire Wire Line
-	3000 2450 3000 2500
+	2150 2450 3200 2450
+Wire Wire Line
+	2450 2450 2450 2500
 Wire Wire Line
 	4550 2650 4650 2650
@@
 	4650 2650 4650 2850
 Wire Wire Line
-	4550 2750 4950 2750
-Wire Wire Line
-	4850 2750 4850 2850
-Connection ~ 4850 2750
-Wire Wire Line
-	2700 2500 2700 2450
-Connection ~ 3000 2450
-Wire Wire Line
-	2850 2400 2850 2450
-Connection ~ 2850 2450
-Wire Wire Line
-	2700 2900 2700 2950
-Wire Wire Line
-	2700 2950 3000 2950
-Wire Wire Line
-	2850 2950 2850 3000
-Wire Wire Line
-	3000 2950 3000 2900
-Connection ~ 2850 2950
-Wire Wire Line
-	6350 2750 6250 2750
-Wire Wire Line
-	6250 2750 6250 2550
+	4850 2750 4850 3350
+Wire Wire Line
+	2150 2500 2150 2450
+Connection ~ 2450 2450
+Wire Wire Line
+	2300 2400 2300 2450
+Connection ~ 2300 2450
+Wire Wire Line
+	2150 2900 2150 2950
+Wire Wire Line
+	2150 2950 2450 2950
+Wire Wire Line
+	2300 2950 2300 3000
+Wire Wire Line
+	2450 2950 2450 2900
+Connection ~ 2300 2950
 Wire Wire Line
 	4550 2550 6350 2550
 Wire Wire Line
 	6100 2550 6100 2650
-Connection ~ 6250 2550
 Wire Wire Line
 	6300 2550 6300 2200
@@
 	2750 4300 5000 4300
 Wire Wire Line
-	3350 2750 3300 2750
+	3000 2750 3350 2750
 Wire Wire Line
 	3300 2750 3300 4200
 Wire Wire Line
 	3300 4200 2750 4200
-Wire Wire Line
-	5800 2650 5800 2550
-Connection ~ 5800 2550
 Wire Wire Line
 	6350 4400 6350 4900
@@
 Wire Wire Line
 	6750 4300 6800 4300
-Text Label 5200 2550 0    39   ~ 0
+Text Label 4750 2550 0    39   ~ 0
 +5V_Gated
 Text Label 7350 2200 0    39   ~ 0
@@
 $EndComp
 Connection ~ 2950 4400
+$Comp
+L R R6
+U 1 1 536DB50B
+P 3000 3050
+F 0 "R6" V 3080 3050 40  0000 C CNN
+F 1 "100K" V 3007 3051 40  0000 C CNN
+F 2 "~" V 2930 3050 30  0000 C CNN
+F 3 "~" H 3000 3050 30  0000 C CNN
+	1    3000 3050
+	1    0    0    -1
+$EndComp
+Wire Wire Line
+	3000 2800 3000 2750
+Connection ~ 3300 2750
+$Comp
+L GND #PWR021
+U 1 1 536DB5BC
+P 3000 3300
+F 0 "#PWR021" H 3000 3300 30  0001 C CNN
+F 1 "GND" H 3000 3230 30  0001 C CNN
+F 2 "" H 3000 3300 60  0000 C CNN
+F 3 "" H 3000 3300 60  0000 C CNN
+	1    3000 3300
+	1    0    0    -1
+$EndComp
+Wire Wire Line
+	4850 3350 6300 3350
+Wire Wire Line
+	6300 3350 6300 2750
+Wire Wire Line
+	6300 2750 6350 2750
+Wire Wire Line
+	4850 2750 4550 2750
+Wire Wire Line
+	5450 2750 5450 2800
+Wire Wire Line
+	5450 3300 5450 3350
+Connection ~ 5450 3350
 $EndSCHEMATC

Commit message: 0.8.0, imported from xwhatits untracked repository
Parts:
- D1: value 1N5819 -> B220A
- D2: value LED -> Actuating
Changed lines of the file:
@@
 Sheet 1 1
 Title "noname.sch"
-Date "10 may 2014"
+Date "11 aug 2014"
 Rev ""
 Comp ""
@@
 P 6550 4300
 F 0 "D2" H 6550 4400 50  0000 C CNN
-F 1 "LED" H 6550 4200 50  0000 C CNN
+F 1 "Actuating" H 6550 4200 50  0000 C CNN
 F 2 "~" H 6550 4300 60  0000 C CNN
 F 3 "~" H 6550 4300 60  0000 C CNN
@@
 P 7850 2550
 F 0 "D1" H 7850 2650 40  0000 C CNN
-F 1 "1N5819" H 7850 2450 40  0000 C CNN
+F 1 "B220A" H 7850 2450 40  0000 C CNN
 F 2 "~" H 7850 2550 60  0000 C CNN
 F 3 "~" H 7850 2550 60  0000 C CNN
